File: hardware/Main.sch (EAGLE design)
At the start: 43 parts, among them IC1 4051N, IC10 L293D, IC11 L293D, IC12 M74HC238, IC13 M74HC238, IC14 74AS08N, IC15 M74HC238, IC16 M74HC238, IC17 MPR121 (0x5A), IC18 MPR121 (0x5B), IC2 4051N, IC3 L293D, IC4 L293D, IC5 L293D, IC6 L293D, IC7 L293D, IC8 L293D, IC9 L293D

Commit message: Removed wrong headers, fixed V33 vs VCC mapping
Parts:
- removed SV1, SV10, SV11, SV12, SV13, SV14, SV15, SV16, SV17, SV2, SV3, SV4, SV5, SV6, SV7, SV8, SV9: (no value), con-dil:28P
- added JP1: (no value), pinhead:PINHD-2X4
Connections:
- removed net F+: SV1.4, SV10.4, SV11.4, SV12.4, SV13.4, SV14.4, SV15.4, SV16.4, SV17.4, SV2.4, SV3.4, SV4.4, SV5.4, SV6.4, SV7.4, SV8.4, SV9.4
- removed net F-: SV1.3, SV10.3, SV11.3, SV12.3, SV13.3, SV14.3, SV15.3, SV16.3, SV17.3, SV2.3, SV3.3, SV4.3, SV5.3, SV6.3, SV7.3, SV8.3, SV9.3
- removed net F0L1-: SV1.25
- removed net F0L1B: SV1.24
- removed net F0L1G: SV1.23
- removed net F0L1R: SV1.26
- removed net F0L2-: SV1.19
- removed net F0L2B: SV1.18
- removed net F0L2G: SV1.17
- removed net F0L2R: SV1.20
- removed net F0S1A: SV1.27
- removed net F0S1B: SV1.28
- removed net F0S2A: SV1.21
- removed net F0S2B: SV1.22
- removed net F10L1-: SV11.25
- removed net F10L1B: SV11.24
- removed net F10L1G: SV11.23
- removed net F10L1R: SV11.26
- removed net F10L2-: SV11.19
- removed net F10L2B: SV11.18
- removed net F10L2G: SV11.17
- removed net F10L2R: SV11.20
- removed net F10S1A: SV11.27
- removed net F10S1B: SV11.28
- removed net F10S2A: SV11.21
- removed net F10S2B: SV11.22
- removed net F11L1-: SV12.25
- removed net F11L1B: SV12.24
- removed net F11L1G: SV12.23
- removed net F11L1R: SV12.26
- removed net F11L2-: SV12.19
- removed net F11L2B: SV12.18
- removed net F11L2G: SV12.17
- removed net F11L2R: SV12.20
- removed net F11S1A: SV12.27
- removed net F11S1B: SV12.28
- removed net F11S2A: SV12.21
- removed net F11S2B: SV12.22
- removed net F12L1-: SV13.25
- removed net F12L1B: SV13.24
- removed net F12L1G: SV13.23
- removed net F12L1R: SV13.26
- removed net F12L2-: SV13.19
- removed net F12L2B: SV13.18
- removed net F12L2G: SV13.17
- removed net F12L2R: SV13.20
- removed net F12S1A: SV13.27
- removed net F12S1B: SV13.28
- removed net F12S2A: SV13.21
- removed net F12S2B: SV13.22
- removed net F13L1-: SV14.25
- removed net F13L1B: SV14.24
- removed net F13L1G: SV14.23
- removed net F13L1R: SV14.26
- removed net F13L2-: SV14.19
- removed net F13L2B: SV14.18
- removed net F13L2G: SV14.17
- removed net F13L2R: SV14.20
- removed net F13S1A: SV14.27
- removed net F13S1B: SV14.28
- removed net F13S2A: SV14.21
- removed net F13S2B: SV14.22
- removed net F14L1-: SV15.25
- removed net F14L1B: SV15.24
- removed net F14L1G: SV15.23
- removed net F14L1R: SV15.26
- removed net F14L2-: SV15.19
- removed net F14L2B: SV15.18
- removed net F14L2G: SV15.17
- removed net F14L2R: SV15.20
- removed net F14S1A: SV15.27
- removed net F14S1B: SV15.28
- removed net F14S2A: SV15.21
- removed net F14S2B: SV15.22
- removed net F15L1-: SV16.25
- removed net F15L1B: SV16.24
- removed net F15L1G: SV16.23
- removed net F15L1R: SV16.26
- removed net F15L2-: SV16.19
- removed net F15L2B: SV16.18
- removed net F15L2G: SV16.17
- removed net F15L2R: SV16.20
- removed net F15S1A: SV16.27
- removed net F15S1B: SV16.28
- removed net F15S2A: SV16.21
- removed net F15S2B: SV16.22
- removed net F1L1-: SV2.25
- removed net F1L1B: SV2.24
- removed net F1L1G: SV2.23
- removed net F1L1R: SV2.26
- removed net F1L2-: SV2.19
- removed net F1L2B: SV2.18
- removed net F1L2G: SV2.17
- removed net F1L2R: SV2.20
- removed net F1S1A: SV2.27
- removed net F1S1B: SV2.28
- removed net F1S2A: SV2.21
- removed net F1S2B: SV2.22
- removed net F2L1-: SV3.25
- removed net F2L1B: SV3.24
- removed net F2L1G: SV3.23
- removed net F2L1R: SV3.26
- removed net F2L2-: SV3.19
- removed net F2L2B: SV3.18
- removed net F2L2G: SV3.17
- removed net F2L2R: SV3.20
- removed net F2S1A: SV3.27
- removed net F2S1B: SV3.28
- removed net F2S2A: SV3.21
- removed net F2S2B: SV3.22
- removed net F3L1-: SV4.25
- removed net F3L1B: SV4.24
- removed net F3L1G: SV4.23
- removed net F3L1R: SV4.26
- removed net F3L2-: SV4.19
- removed net F3L2B: SV4.18
- removed net F3L2G: SV4.17
- removed net F3L2R: SV4.20
- removed net F3S1A: SV4.27
- removed net F3S1B: SV4.28
- removed net F3S2A: SV4.21
- removed net F3S2B: SV4.22
- removed net F4L1-: SV5.25
- removed net F4L1B: SV5.24
- removed net F4L1G: SV5.23
- removed net F4L1R: SV5.26
- removed net F4L2-: SV5.19
- removed net F4L2B: SV5.18
- removed net F4L2G: SV5.17
- removed net F4L2R: SV5.20
- removed net F4S1A: SV5.27
- removed net F4S1B: SV5.28
- removed net F4S2A: SV5.21
- removed net F4S2B: SV5.22
- removed net F5L1-: SV6.25
- removed net F5L1B: SV6.24
- removed net F5L1G: SV6.23
- removed net F5L1R: SV6.26
- removed net F5L2-: SV6.19
- removed net F5L2B: SV6.18
- removed net F5L2G: SV6.17
- removed net F5L2R: SV6.20
- removed net F5S1A: SV6.27
- removed net F5S1B: SV6.28
- removed net F5S2A: SV6.21
- removed net F5S2B: SV6.22
- removed net F6L1-: SV7.25
- removed net F6L1B: SV7.24
- removed net F6L1G: SV7.23
- removed net F6L1R: SV7.26
- removed net F6L2-: SV7.19
- removed net F6L2B: SV7.18
- removed net F6L2G: SV7.17
- removed net F6L2R: SV7.20
- removed net F6S1A: SV7.27
- removed net F6S1B: SV7.28
- removed net F6S2A: SV7.21
- removed net F6S2B: SV7.22
- removed net F7L1-: SV8.25
- removed net F7L1B: SV8.24
- removed net F7L1G: SV8.23
- removed net F7L1R: SV8.26
- removed net F7L2-: SV8.19
- removed net F7L2B: SV8.18
- removed net F7L2G: SV8.17
- removed net F7L2R: SV8.20
- removed net F7S1A: SV8.27
- removed net F7S1B: SV8.28
- removed net F7S2A: SV8.21
- removed net F7S2B: SV8.22
- removed net F8L1-: SV9.25
- removed net F8L1B: SV9.24
- removed net F8L1G: SV9.23
- removed net F8L1R: SV9.26
- removed net F8L2-: SV9.19
- removed net F8L2B: SV9.18
- removed net F8L2G: SV9.17
- removed net F8L2R: SV9.20
- removed net F8S1A: SV9.27
- removed net F8S1B: SV9.28
- removed net F8S2A: SV9.21
- removed net F8S2B: SV9.22
- removed net F9L1-: SV10.25
- removed net F9L1B: SV10.24
- removed net F9L1G: SV10.23
- removed net F9L1R: SV10.26
- removed net F9L2-: SV10.19
- removed net F9L2B: SV10.18
- removed net F9L2G: SV10.17
- removed net F9L2R: SV10.20
- removed net F9S1A: SV10.27
- removed net F9S1B: SV10.28
- removed net F9S2A: SV10.21
- removed net F9S2B: SV10.22
- removed net N$3: C3.2
- removed net SSGND: SV1.15, SV10.15, SV11.15, SV12.15, SV13.15, SV14.15, SV15.15, SV16.15, SV2.15, SV3.15, SV4.15, SV5.15, SV6.15, SV7.15, SV8.15, SV9.15
- removed net SSVCC: SV1.9, SV10.9, SV11.9, SV12.9, SV13.9, SV14.9, SV15.9, SV16.9, SV2.9, SV3.9, SV4.9, SV5.9, SV6.9, SV7.9, SV8.9, SV9.9
- removed net VCC_2: B1.AREF, C2.1, C4.1, IC17.VSS, IC18.ADDR, IC18.VSS
- new net VREF: B1.AREF, JP1.7
- net A2: no longer SV17.5
- net F0: no longer SV1.5
- net F1: no longer SV2.5
- net F10: no longer SV11.5
- net F11: no longer SV12.5
- net F12: no longer SV13.5
- net F13: no longer SV14.5
- net F14: no longer SV15.5
- net F15: no longer SV16.5
- net F2: no longer SV3.5
- net F3: no longer SV4.5
- net F4: no longer SV5.5
- net F5: no longer SV6.5
- net F6: no longer SV7.5
- net F7: no longer SV8.5
- net F8: no longer SV9.5
- net F9: no longer SV10.5
- net FMOT0+: no longer SV1.1
- net FMOT0-: no longer SV1.2
- net FMOT1+: no longer SV2.1
- net FMOT1-: no longer SV2.2
- net FMOT10+: no longer SV11.1
- net FMOT10-: no longer SV11.2
- net FMOT11+: no longer SV12.1
- net FMOT11-: no longer SV12.2
- net FMOT12+: no longer SV13.1
- net FMOT12-: no longer SV13.2
- net FMOT13+: no longer SV14.1
- net FMOT13-: no longer SV14.2
- net FMOT14+: no longer SV15.1
- net FMOT14-: no longer SV15.2
- net FMOT15+: no longer SV16.1
- net FMOT15-: no longer SV16.2
- net FMOT2+: no longer SV3.1
- net FMOT2-: no longer SV3.2
- net FMOT3+: no longer SV4.1
- net FMOT3-: no longer SV4.2
- net FMOT4+: no longer SV5.1
- net FMOT4-: no longer SV5.2
- net FMOT5+: no longer SV6.1
- net FMOT5-: no longer SV6.2
- net FMOT6+: no longer SV7.1
- net FMOT6-: no longer SV7.2
- net FMOT7+: no longer SV8.1
- net FMOT7-: no longer SV8.2
- net FMOT8+: no longer SV9.1
- net FMOT8-: no longer SV9.2
- net FMOT9+: no longer SV10.1
- net FMOT9-: no longer SV10.2
- net FMOTM+: no longer SV17.1
- net FMOTM-: no longer SV17.2
- net FT0: no longer SV1.8
- net FT1: no longer SV2.8
- net FT10: no longer SV11.8
- net FT11: no longer SV12.8
- net FT12: no longer SV13.8
- net FT13: no longer SV14.8
- net FT14: no longer SV15.8
- net FT15: no longer SV16.8
- net FT2: no longer SV3.8
- net FT3: no longer SV4.8
- net FT4: no longer SV5.8
- net FT5: no longer SV6.8
- net FT6: no longer SV7.8
- net FT7: no longer SV8.8
- net FT8: no longer SV9.8
- net FT9: no longer SV10.8
- net FTM: no longer SV17.8
- net GND: now also C3.2, JP1.1, JP1.8; no longer SV1.10, SV1.6, SV1.7, SV10.10, SV10.6, SV10.7, SV11.10, SV11.6, SV11.7, SV12.10, SV12.6, SV12.7, SV13.10, SV13.6, SV13.7, SV14.10, SV14.6, SV14.7, SV15.10, SV15.6, SV15.7, SV16.10, SV16.6, SV16.7, SV17.10, SV17.6, SV17.7, SV2.10, SV2.6, SV2.7, SV3.10, SV3.6, SV3.7, SV4.10, SV4.6, SV4.7, SV5.10, SV5.6, SV5.7, SV6.10, SV6.6, SV6.7, SV7.10, SV7.6, SV7.7, SV8.10, SV8.6, SV8.7, SV9.10, SV9.6, SV9.7
- net SSCLK: now also JP1.5; no longer SV1.13, SV10.13, SV11.13, SV12.13, SV13.13, SV14.13, SV15.13, SV16.13, SV2.13, SV3.13, SV4.13, SV5.13, SV6.13, SV7.13, SV8.13, SV9.13
- net SSCS0: no longer SV1.12
- net SSCS1: no longer SV2.12
- net SSCS10: no longer SV11.12
- net SSCS11: no longer SV12.12
- net SSCS12: no longer SV13.12
- net SSCS13: no longer SV14.12
- net SSCS14: no longer SV15.12
- net SSCS15: no longer SV16.12
- net SSCS2: no longer SV3.12
- net SSCS3: no longer SV4.12
- net SSCS4: no longer SV5.12
- net SSCS5: no longer SV6.12
- net SSCS6: no longer SV7.12
- net SSCS7: no longer SV8.12
- net SSCS8: no longer SV9.12
- net SSCS9: no longer SV10.12
- net SSDC: now also JP1.4; no longer SV1.14, SV10.14, SV11.14, SV12.14, SV13.14, SV14.14, SV15.14, SV16.14, SV2.14, SV3.14, SV4.14, SV5.14, SV6.14, SV7.14, SV8.14, SV9.14
- net SSMOSI: now also JP1.3; no longer SV1.16, SV10.16, SV11.16, SV12.16, SV13.16, SV14.16, SV15.16, SV16.16, SV2.16, SV3.16, SV4.16, SV5.16, SV6.16, SV7.16, SV8.16, SV9.16
- net SSRST: now also JP1.6; no longer SV1.11, SV10.11, SV11.11, SV12.11, SV13.11, SV14.11, SV15.11, SV16.11, SV2.11, SV3.11, SV4.11, SV5.11, SV6.11, SV7.11, SV8.11, SV9.11
- net V33: now also C2.1, C4.1, IC17.VSS, IC18.ADDR, IC18.VSS
- net VCC: now also JP1.2
Other:
- note added: "F+"
- note added: "F-"
- note removed: "(FM)"

Commit message: Pre-tidy folder structure
Other:
- moved on the sheet: IC10, IC11, IC6, IC7, IC8, IC9, JP1
