File: hardware/board-x8-fader-display/board-x8-fader-display.kicad_pcb (KiCad board)
At the start: 2 copper layers, 41 parts, among them J1 OLED0, J2 OLED1, J3 OLED2, J4 OLED3, J5 OLED4, J6 OLED5, J7 OLED6, J8 OLED7, J9 Conn_02x16_Odd_Even, U1 74xx238, U2 L293, U3 L293, U4 L293, U5 L293, U6 CAP1296, U7 CAP1296, U8 4051, U9 74xx238

Commit message: Adding DIP library for DIP to DFN converter, Updated board layout with autorouting, hopefully v0.1 final design
Parts:
- added REF**: 1pin, Connectors:1pin, F.Cu at (239.5, 235.0)
- added REF**: 1pin, Connectors:1pin, F.Cu at (88.5, 235.0)
- added REF**: 1pin, Connectors:1pin, F.Cu at (180.5, 235.0)
- added REF**: 1pin, Connectors:1pin, F.Cu at (239.5, 75.0)
- added REF**: 1pin, Connectors:1pin, F.Cu at (179.5, 75.0)
- added REF**: 1pin, Connectors:1pin, F.Cu at (324.5, 75.0)
- added REF**: 1pin, Connectors:1pin, F.Cu at (88.5, 75.0)
- added REF**: 1pin, Connectors:1pin, F.Cu at (88.5, 33.0)
- added REF**: 1pin, Connectors:1pin, F.Cu at (330.5, 33.0)
- added REF**: 1pin, Connectors:1pin, F.Cu at (330.5, 235.0)
- C1, C10, C11, C12, C13, C2, C3, C4, C5, C6, C7, C8, C9: footprint Capacitors_SMD:C_0805_HandSoldering -> Capacitors_THT:C_Disc_D5.0mm_W2.5mm_P5.00mm
- R1, R2: footprint Resistors_SMD:R_1206_HandSoldering -> Resistors_THT:R_Axial_DIN0204_L3.6mm_D1.6mm_P5.08mm_Horizontal
- U6, U7: footprint Housings_DFN_QFN:DFN-10-1EP_3x3mm_Pitch0.5mm -> ca_dip:DIP-10_W13.38mm+GND
- moved C5 169.1 mm to (297.5, 186.0)
- moved C12 161.0 mm to (270.0, 82.0), turned to 270 degrees
- moved C11 149.6 mm to (272.5, 138.5)
- moved C2 144.7 mm to (177.5, 186.0)
- moved C3 144.7 mm to (207.5, 186.0)
- moved C4 144.3 mm to (237.0, 186.0)
- moved C1 126.2 mm to (122.5, 186.0), turned to 180 degrees
- moved C8 95.9 mm to (150.0, 82.0), turned to 270 degrees
- moved U8 82.4 mm to (213.5, 128.1), turned to 180 degrees
- moved U6 80.1 mm to (157.0, 122.0), turned to 180 degrees
- moved U7 79.5 mm to (276.4, 122.1), turned to 180 degrees
- moved C10 74.0 mm to (182.5, 221.5)
- moved C9 73.9 mm to (122.5, 221.5)
- moved C13 73.6 mm to (302.5, 221.5), turned to 180 degrees
- moved U1 71.4 mm to (200.9, 78.6)
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Connections:
- J1 pad 1: Net-(J1-Pad1) -> GND
- J1 pad 2: Net-(J1-Pad2) -> VCC
- J2 pad 1: Net-(J1-Pad1) -> GND
- J2 pad 2: Net-(J1-Pad2) -> VCC
- J3 pad 1: Net-(J1-Pad1) -> GND
- J3 pad 2: Net-(J1-Pad2) -> VCC
- J4 pad 1: Net-(J1-Pad1) -> GND
- J4 pad 2: Net-(J1-Pad2) -> VCC
- J5 pad 1: Net-(J1-Pad1) -> GND
- J5 pad 2: Net-(J1-Pad2) -> VCC
- J6 pad 1: Net-(J1-Pad1) -> GND
- J6 pad 2: Net-(J1-Pad2) -> VCC
- J7 pad 1: Net-(J1-Pad1) -> GND
- J7 pad 2: Net-(J1-Pad2) -> VCC
- J8 pad 1: Net-(J1-Pad1) -> GND
- J8 pad 2: Net-(J1-Pad2) -> VCC
- U6 pad 1: (no net) -> /FCAP0
- U6 pad 10: GND -> /FCAP1
- U6 pad 11: /FCAP3 -> GND
- U6 pad 2: /FCAP0 -> Net-(R1-Pad1)
- U6 pad 3: Net-(R1-Pad1) -> /FSDAa
- U6 pad 4: /FSDAa -> /FSCLa
- U6 pad 5: /FSCLa -> VCC
- U6 pad 6: (no net) -> GND
- U6 pad 7: VCC -> GND
- U6 pad 8: GND -> /FCAP3
- U6 pad 9: GND -> /FCAP2
- U7 pad 1: (no net) -> /FCAP4
- U7 pad 10: GND -> /FCAP5
- U7 pad 11: /FCAP7 -> GND
- U7 pad 2: /FCAP4 -> Net-(R2-Pad1)
- U7 pad 3: Net-(R2-Pad1) -> /FSDAb
- U7 pad 4: /FSDAb -> /FSCLb
- U7 pad 5: /FSCLb -> VCC
- U7 pad 6: (no net) -> GND
- U7 pad 7: VCC -> GND
- U7 pad 8: GND -> /FCAP7
- U7 pad 9: GND -> /FCAP6
Routing:
- net GND: track 0.00 -> 1230.5 mm
- net VCC: track 0.00 -> 918.5 mm, vias 0 -> 2
- net /MCTLA: track 0.00 -> 386.4 mm, vias 0 -> 2
- net /DDC: track 0.00 -> 375.7 mm, vias 0 -> 7
- net /D~RST~: track 0.00 -> 367.3 mm, vias 0 -> 1
- net /MCTLB: track 0.00 -> 340.7 mm, vias 0 -> 2
- net +12V: track 0.00 -> 318.7 mm
- net VREF: track 0.00 -> 272.1 mm
- net /FSCL: track 0.00 -> 241.8 mm, vias 0 -> 3
- net /FSDA: track 0.00 -> 234.0 mm
- net /DA2: track 0.00 -> 203.8 mm
- net /FSDAa: track 0.00 -> 191.4 mm
- net /FSCLa: track 0.00 -> 185.5 mm
- net /DA0: track 0.00 -> 178.4 mm, vias 0 -> 1
- net /DA1: track 0.00 -> 165.6 mm, vias 0 -> 1
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Other:
- board outline added: 250 x 210 mm
- net class Default: clearance 0.2 -> 0.5; trace_width 0.25 -> 0.6; via_dia 0.6 -> 0.8; via_drill 0.4 -> 0.6
- net class Power added: clearance 0.5, trace_width 1, via_dia 1.2, via_drill 1
- rule trace_clearance: 0.2 -> 0.5
- board text added: "Faderboard v0.1 C Ashby 17-MAY-2018"
