File: hardware/board-x8-fader-display/board-x8-fader-display.kicad_pcb (KiCad board)
At the start: 2 copper layers, 250 x 210 mm, 51 parts, among them J1 OLED0, J2 OLED1, J3 OLED2, J4 OLED3, J5 OLED4, J6 OLED5, J7 OLED6, J8 OLED7, J9 Conn_02x16_Odd_Even, U1 74xx238, U2 L293, U3 L293, U4 L293, U5 L293, U6 CAP1296, U7 CAP1296, U8 4051, U9 74xx238

Commit message: Snagging complete on Schematic - PCB still out of date
Parts:
- renumbered REF** to REF1, REF** to REF10, REF** to REF2, REF** to REF3, REF** to REF4, REF** to REF5, REF** to REF6, REF** to REF7, REF** to REF8, REF** to REF9
Routing:
- net GND: track 1230.5 -> 1316.8 mm, vias 0 -> 2
- net /FA3: track 159.5 -> 120.6 mm, vias 1 -> 2
- net /DA2: track 203.8 -> 172.8 mm, vias 0 -> 2
- net /MCTLA: track 386.4 -> 358.8 mm, vias 2 -> 3
- net VCC: track 918.5 -> 895.9 mm
- net VREF: track 272.1 -> 293.3 mm, vias 0 -> 1
- net /FCAP6: track 37.5 -> 58.7 mm
- net /FCAP3: track 68.9 -> 85.9 mm
- net /FSDAb: track 77.8 -> 63.0 mm, vias 1 -> 0
- net /MEN5: track 69.5 -> 55.2 mm, vias 0 -> 1
- net /FSDAa: track 191.4 -> 178.0 mm, vias 0 -> 2
- net /MEN0: track 126.7 -> 113.9 mm
- net /DA1: track 165.6 -> 153.3 mm
- net /DA3: track 153.4 -> 142.2 mm, vias 1 -> 0
- net /FA1: track 145.0 -> 134.2 mm, vias 0 -> 1
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Other:
- outline, holes or cut-outs redrawn

Commit message: Updated with new DRSTx functionality, Updated silkscreen for fader to include cut slot and screws (for use with panel cutter), Still need to modify display silkscreen, Sanitised .gitignore
Parts:
- removed R1, R2: 2k2, Resistors_THT:R_Axial_DIN0204_L3.6mm_D1.6mm_P5.08mm_Horizontal
- added U2: 74xx138, Housings_DIP:DIP-16_W7.62mm, F.Cu at (261.5, 79.0)
- J9: moved to B.Cu
- U1: value 74xx238 -> 74xx138
- moved U1 59.4 mm to (141.5, 80.0)
- moved J9 11.8 mm to (322.5, 133.0), turned to 180 degrees
- moved U8 5.92 mm to (276.5, 128.0)
- moved C8 5.02 mm to (149.5, 87.0)
- moved U7 5.02 mm to (156.5, 127.0)
- moved C12 4.03 mm to (269.5, 86.0)
- renumbered U9 to U10, U2 to U3, U3 to U4, U4 to U5, U5 to U6, U6 to U7, U7 to U8, U8 to U9
Connections:
- net /DCS0 renamed /D~CS~0
- net /DCS1 renamed /D~CS~1
- net /DCS2 renamed /D~CS~2
- net /DCS3 renamed /D~CS~3
- net /DCS4 renamed /D~CS~4
- net /DCS5 renamed /D~CS~5
- net /DCS6 renamed /D~CS~6
- net /DCS7 renamed /D~CS~7
- J1 pad 3: /FSCL -> /DSCL
- J1 pad 4: /FSDA -> /DSDA
- J1 pad 5: /D~RST~ -> /D~RST~0
- J2 pad 3: /FSCL -> /DSCL
- J2 pad 4: /FSDA -> /DSDA
- J2 pad 5: /D~RST~ -> /D~RST~1
- J3 pad 3: /FSCL -> /DSCL
- J3 pad 4: /FSDA -> /DSDA
- J3 pad 5: /D~RST~ -> /D~RST~2
- J4 pad 3: /FSCL -> /DSCL
- J4 pad 4: /FSDA -> /DSDA
- J4 pad 5: /D~RST~ -> /D~RST~3
- J5 pad 3: /FSCL -> /DSCL
- J5 pad 4: /FSDA -> /DSDA
- J5 pad 5: /D~RST~ -> /D~RST~4
- J6 pad 3: /FSCL -> /DSCL
- J6 pad 4: /FSDA -> /DSDA
- J6 pad 5: /D~RST~ -> /D~RST~5
- J7 pad 3: /FSCL -> /DSCL
- J7 pad 4: /FSDA -> /DSDA
- J7 pad 5: /D~RST~ -> /D~RST~6
- J8 pad 3: /FSCL -> /DSCL
- J8 pad 4: /FSDA -> /DSDA
- J8 pad 5: /D~RST~ -> /D~RST~7
- J9 pad 11: GND -> /F~INT~a
- J9 pad 12: /F~IRQ~ -> /BSEL
- J9 pad 17: /MA1 -> /F~INT~b
- J9 pad 18: /MA2 -> /MA1
- J9 pad 19: /MA3 -> /MA2
- J9 pad 23: /FA3 -> GND
- J9 pad 27: /DA3 -> GND
- J9 pad 28: /D~RST~ -> /DSDA
- J9 pad 30: /BSEL -> /DSCL
- J9 pad 31: GND -> /D~CS~
- J9 pad 32: GND -> /D~RST~
- U1 pad 5: GND -> /D~CS~
- U1 pad 6: /DA3 -> /BSEL
- U10 pad 6: /MA3 -> /BSEL
- U7 pad 2: Net-(R1-Pad1) -> /F~INT~a
- U8 pad 2: Net-(R2-Pad1) -> /F~INT~b
- U9 pad 6: /FA3 -> /BSEL
Routing:
- net /DSDA: track 0.00 -> 405.5 mm, vias 0 -> 1
- net /DSCL: track 0.00 -> 376.1 mm, vias 0 -> 2
- net /BSEL: track 0.00 -> 353.2 mm, vias 0 -> 2
- net /FSCL: track 240.7 -> 0.00 mm, vias 3 -> 0
- net /D~RST~: track 357.0 -> 117.0 mm, vias 2 -> 0
- net /FSDA: track 239.1 -> 0.00 mm, vias 2 -> 0
- net /D~CS~: track 0.00 -> 224.2 mm, vias 0 -> 2
- net /F~INT~a: track 0.00 -> 210.6 mm
- net /D~RST~0: track 0.00 -> 170.5 mm, vias 0 -> 1
- net /D~RST~1: track 0.00 -> 144.4 mm, vias 0 -> 1
- net /DA3: track 142.2 -> 0.00 mm
- net /MA3: track 130.2 -> 0.00 mm, vias 1 -> 0
- net /FA3: track 120.6 -> 0.00 mm, vias 2 -> 0
- net /D~RST~2: track 0.00 -> 115.5 mm
- net /DA1: track 153.3 -> 265.8 mm, vias 1 -> 2
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Other:
- net class Default: trace_width 0.6 -> 0.5
- rule trace_min: 0.2 -> 0.125

Commit message: Updated displays with silkscreen additions for cutouts, Updated PCB latest version (NOTE may need to change CAP1296 DFN to DIP adaptor depending on recent purchase / availability
Routing:
- net GND: track 1368.8 -> 0.00 mm, vias 1 -> 0
- net VCC: track 948.5 -> 0.00 mm
- net /DSDA: track 405.5 -> 0.00 mm, vias 1 -> 0
- net /MCTLB: track 385.6 -> 0.00 mm, vias 3 -> 0
- net /DSCL: track 376.1 -> 0.00 mm, vias 2 -> 0
- net /DDC: track 371.0 -> 0.00 mm, vias 4 -> 0
- net /BSEL: track 353.2 -> 0.00 mm, vias 2 -> 0
- net /MCTLA: track 338.2 -> 0.00 mm, vias 3 -> 0
- net +12V: track 323.2 -> 0.00 mm, vias 2 -> 0
- net VREF: track 278.2 -> 0.00 mm
- net /DA1: track 265.8 -> 0.00 mm, vias 2 -> 0
- net /DA0: track 249.5 -> 0.00 mm, vias 1 -> 0
- net /DA2: track 245.4 -> 0.00 mm, vias 1 -> 0
- net /D~CS~: track 224.2 -> 0.00 mm, vias 2 -> 0
- net /F~INT~a: track 210.6 -> 0.00 mm
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
Commit message: Updating PCB and schema for ProtoAdvantage DIP to DFN adapter (not great but easier than SMD on this board). Rerouting and manual edits to conform to DRC / track & pad clearance
Parts:
- U7, U8: footprint ca_dip:DIP-10_W13.38mm+GND -> ca_dip:PROTOADVANTAGE_DIPDFN10_3x3
- moved U8 11.5 mm to (270.2, 118.4), turned to 90 degrees
- moved U7 10.8 mm to (150.0, 118.4), turned to 90 degrees
Connections:
- J9 pad 4: GND -> +12V
Routing:
- net GND: track 0.00 -> 1325.4 mm
- net VCC: track 0.00 -> 959.2 mm, vias 0 -> 1
- net /DSCL: track 0.00 -> 381.4 mm
- net /DSDA: track 0.00 -> 379.1 mm, vias 0 -> 1
- net /DDC: track 0.00 -> 376.4 mm, vias 0 -> 3
- net /MCTLA: track 0.00 -> 337.5 mm, vias 0 -> 4
- net /MCTLB: track 0.00 -> 331.4 mm, vias 0 -> 2
- net /BSEL: track 0.00 -> 330.2 mm, vias 0 -> 2
- net +12V: track 0.00 -> 310.7 mm, vias 0 -> 2
- net VREF: track 0.00 -> 277.0 mm
- net /DA1: track 0.00 -> 258.3 mm, vias 0 -> 1
- net /DA0: track 0.00 -> 239.6 mm, vias 0 -> 1
- net /DA2: track 0.00 -> 235.8 mm, vias 0 -> 1
- net /FSDAa: track 0.00 -> 234.8 mm
- net /FSCLa: track 0.00 -> 231.5 mm
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- added copper zone on B.Cu, net GND
- added copper zone on F.Cu, net GND
