File: hardware/board-x8-fader-display/board-x8-fader-display.sch (KiCad schematic (older format))
At the start: 41 parts, among them J1 OLED0, J2 OLED1, J3 OLED2, J4 OLED3, J5 OLED4, J6 OLED5, J7 OLED6, J8 OLED7, J9 Conn_02x16_Odd_Even, U1 74xx238, U2 L293, U3 L293, U4 L293, U5 L293, U6 CAP1296, U7 CAP1296, U8 4051, U9 74xx238

Commit message: Adding Fader data sheet, Schema v1 for faders complete, starting to get footprints sorted out
Parts:
- C1, C10, C11, C12, C13, C2, C3, C4, C5, C6, C7, C8, C9: footprint (none) -> Capacitors_SMD:C_0805_HandSoldering
- J1, J2, J3, J4, J5, J6, J7, J8: footprint (none) -> Socket_Strips:Socket_Strip_Straight_1x07
- J9: footprint (none) -> Pin_Headers:Pin_Header_Straight_2x16
- R1, R2: footprint (none) -> Resistors_SMD:R_1206_HandSoldering
- RV1, RV2, RV3, RV4, RV5, RV6, RV7, RV8: footprint (none) -> ca_alps:AlpsFader_RSA0N11M9A0J
- U1, U2, U3, U4, U5, U8, U9: footprint (none) -> Housings_DIP:DIP-16_W7.62mm
- U6, U7: footprint (none) -> Housings_DFN_QFN:DFN-10-1EP_3x3mm_Pitch0.5mm
Changed lines of the file:
@@
 F 0 "RV1" H 6150 1850 50  0000 C CNN
 F 1 "RSA0N11M9A0J" V 5900 1750 50  0001 C CNN
-F 2 "" H 6000 1750 50  0001 C CNN
+F 2 "ca_alps:AlpsFader_RSA0N11M9A0J" H 6000 1750 50  0001 C CNN
 F 3 "" H 6000 1750 50  0001 C CNN
 	1    6000 1750
@@
 F 0 "RV2" H 6150 2600 50  0000 C CNN
 F 1 "RSA0N11M9A0J" V 5900 2500 50  0001 C CNN
-F 2 "" H 6000 2500 50  0001 C CNN
+F 2 "ca_alps:AlpsFader_RSA0N11M9A0J" H 6000 2500 50  0001 C CNN
 F 3 "" H 6000 2500 50  0001 C CNN
 	1    6000 2500
@@
 F 0 "RV3" H 6150 3350 50  0000 C CNN
 F 1 "RSA0N11M9A0J" V 5900 3250 50  0001 C CNN
-F 2 "" H 6000 3250 50  0001 C CNN
+F 2 "ca_alps:AlpsFader_RSA0N11M9A0J" H 6000 3250 50  0001 C CNN
 F 3 "" H 6000 3250 50  0001 C CNN
 	1    6000 3250
@@
 F 0 "RV5" H 6150 4850 50  0000 C CNN
 F 1 "RSA0N11M9A0J" V 5900 4750 50  0001 C CNN
-F 2 "" H 6000 4750 50  0001 C CNN
+F 2 "ca_alps:AlpsFader_RSA0N11M9A0J" H 6000 4750 50  0001 C CNN
 F 3 "" H 6000 4750 50  0001 C CNN
 	1    6000 4750
@@
 F 0 "RV6" H 6150 5600 50  0000 C CNN
 F 1 "RSA0N11M9A0J" V 5900 5500 50  0001 C CNN
-F 2 "" H 6000 5500 50  0001 C CNN
+F 2 "ca_alps:AlpsFader_RSA0N11M9A0J" H 6000 5500 50  0001 C CNN
 F 3 "" H 6000 5500 50  0001 C CNN
 	1    6000 5500
@@
 F 0 "RV7" H 6150 6350 50  0000 C CNN
 F 1 "RSA0N11M9A0J" V 5900 6250 50  0001 C CNN
-F 2 "" H 6000 6250 50  0001 C CNN
+F 2 "ca_alps:AlpsFader_RSA0N11M9A0J" H 6000 6250 50  0001 C CNN
 F 3 "" H 6000 6250 50  0001 C CNN
 	1    6000 6250
@@
 F 0 "RV8" H 6150 7100 50  0000 C CNN
 F 1 "RSA0N11M9A0J" V 5900 7000 50  0001 C CNN
-F 2 "" H 6000 7000 50  0001 C CNN
+F 2 "ca_alps:AlpsFader_RSA0N11M9A0J" H 6000 7000 50  0001 C CNN
 F 3 "" H 6000 7000 50  0001 C CNN
 	1    6000 7000
@@
 F 0 "U8" H 7700 1900 50  0000 C CNN
 F 1 "4051" H 7700 1700 50  0000 C CNN
-F 2 "" H 7600 1900 60  0001 C CNN
+F 2 "Housings_DIP:DIP-16_W7.62mm" H 7600 1900 60  0001 C CNN
 F 3 "" H 7600 1900 60  0001 C CNN
 	1    7600 1900
@@
 F 0 "U2" H 4700 2550 60  0000 C CNN
 F 1 "L293" H 4700 1700 60  0000 C CNN
-F 2 "" H 4650 1800 60  0001 C CNN
+F 2 "Housings_DIP:DIP-16_W7.62mm" H 4650 1800 60  0001 C CNN
 F 3 "" H 4650 1800 60  0001 C CNN
 	1    4700 2100
@@
 F 0 "U3" H 4700 4100 60  0000 C CNN
 F 1 "L293" H 4700 3250 60  0000 C CNN
-F 2 "" H 4650 3350 60  0001 C CNN
+F 2 "Housings_DIP:DIP-16_W7.62mm" H 4650 3350 60  0001 C CNN
 F 3 "" H 4650 3350 60  0001 C CNN
 	1    4700 3650
@@
 F 0 "U5" H 4700 7050 60  0000 C CNN
 F 1 "L293" H 4700 6200 60  0000 C CNN
-F 2 "" H 4650 6300 60  0001 C CNN
+F 2 "Housings_DIP:DIP-16_W7.62mm" H 4650 6300 60  0001 C CNN
 F 3 "" H 4650 6300 60  0001 C CNN
 	1    4700 6600
@@
 F 0 "U4" H 4700 5550 60  0000 C CNN
 F 1 "L293" H 4700 4700 60  0000 C CNN
-F 2 "" H 4650 4800 60  0001 C CNN
+F 2 "Housings_DIP:DIP-16_W7.62mm" H 4650 4800 60  0001 C CNN
 F 3 "" H 4650 4800 60  0001 C CNN
 	1    4700 5100
@@
 F 0 "C2" H 9260 3820 50  0000 L CNN
 F 1 "10nF" H 9260 3670 50  0000 L CNN
-F 2 "" H 9250 3750 50  0001 C CNN
+F 2 "Capacitors_SMD:C_0805_HandSoldering" H 9250 3750 50  0001 C CNN
 F 3 "" H 9250 3750 50  0001 C CNN
 	1    9250 3750
@@
 F 0 "C3" H 9510 3820 50  0000 L CNN
 F 1 "10nF" H 9510 3670 50  0000 L CNN
-F 2 "" H 9500 3750 50  0001 C CNN
+F 2 "Capacitors_SMD:C_0805_HandSoldering" H 9500 3750 50  0001 C CNN
 F 3 "" H 9500 3750 50  0001 C CNN
 	1    9500 3750
@@
 F 0 "C4" H 9760 3820 50  0000 L CNN
 F 1 "10nF" H 9760 3670 50  0000 L CNN
-F 2 "" H 9750 3750 50  0001 C CNN
+F 2 "Capacitors_SMD:C_0805_HandSoldering" H 9750 3750 50  0001 C CNN
 F 3 "" H 9750 3750 50  0001 C CNN
 	1    9750 3750
@@
 F 0 "C5" H 10010 3820 50  0000 L CNN
 F 1 "10nF" H 10010 3670 50  0000 L CNN
-F 2 "" H 10000 3750 50  0001 C CNN
+F 2 "Capacitors_SMD:C_0805_HandSoldering" H 10000 3750 50  0001 C CNN
 F 3 "" H 10000 3750 50  0001 C CNN
 	1    10000 3750
@@
 F 0 "C6" H 10260 3820 50  0000 L CNN
 F 1 "10nF" H 10260 3670 50  0000 L CNN
-F 2 "" H 10250 3750 50  0001 C CNN
+F 2 "Capacitors_SMD:C_0805_HandSoldering" H 10250 3750 50  0001 C CNN
 F 3 "" H 10250 3750 50  0001 C CNN
 	1    10250 3750
@@
 F 0 "C7" H 10510 3820 50  0000 L CNN
 F 1 "10nF" H 10510 3670 50  0000 L CNN
-F 2 "" H 10500 3750 50  0001 C CNN
+F 2 "Capacitors_SMD:C_0805_HandSoldering" H 10500 3750 50  0001 C CNN
 F 3 "" H 10500 3750 50  0001 C CNN
 	1    10500 3750
@@
 F 0 "C10" H 10760 3820 50  0000 L CNN
 F 1 "10nF" H 10760 3670 50  0000 L CNN
-F 2 "" H 10750 3750 50  0001 C CNN
+F 2 "Capacitors_SMD:C_0805_HandSoldering" H 10750 3750 50  0001 C CNN
 F 3 "" H 10750 3750 50  0001 C CNN
 	1    10750 3750
@@
 F 0 "C8" H 10510 4620 50  0000 L CNN
 F 1 "10nF" H 10510 4470 50  0000 L CNN
-F 2 "" H 10500 4550 50  0001 C CNN
+F 2 "Capacitors_SMD:C_0805_HandSoldering" H 10500 4550 50  0001 C CNN
 F 3 "" H 10500 4550 50  0001 C CNN
 	1    10500 4550
@@
 F 0 "C12" H 11010 4620 50  0000 L CNN
 F 1 "10nF" H 11010 4470 50  0000 L CNN
-F 2 "" H 11000 4550 50  0001 C CNN
+F 2 "Capacitors_SMD:C_0805_HandSoldering" H 11000 4550 50  0001 C CNN
 F 3 "" H 11000 4550 50  0001 C CNN
 	1    11000 4550
@@
 F 0 "C9" H 10510 5720 50  0000 L CNN
 F 1 "10nF" H 10510 5570 50  0000 L CNN
-F 2 "" H 10500 5650 50  0001 C CNN
+F 2 "Capacitors_SMD:C_0805_HandSoldering" H 10500 5650 50  0001 C CNN
 F 3 "" H 10500 5650 50  0001 C CNN
 	1    10500 5650
@@
 F 0 "C13" H 11010 5720 50  0000 L CNN
 F 1 "10nF" H 11010 5570 50  0000 L CNN
-F 2 "" H 11000 5650 50  0001 C CNN
+F 2 "Capacitors_SMD:C_0805_HandSoldering" H 11000 5650 50  0001 C CNN
 F 3 "" H 11000 5650 50  0001 C CNN
 	1    11000 5650
@@
 F 0 "J1" H 650 1400 50  0000 C CNN
 F 1 "OLED0" H 650 600 50  0000 C CNN
-F 2 "" H 650 1000 50  0001 C CNN
+F 2 "Socket_Strips:Socket_Strip_Straight_1x07" H 650 1000 50  0001 C CNN
 F 3 "" H 650 1000 50  0001 C CNN
 	1    650  1000
@@
 F 0 "J2" H 650 2300 50  0000 C CNN
 F 1 "OLED1" H 650 1500 50  0000 C CNN
-F 2 "" H 650 1900 50  0001 C CNN
+F 2 "Socket_Strips:Socket_Strip_Straight_1x07" H 650 1900 50  0001 C CNN
 F 3 "" H 650 1900 50  0001 C CNN
 	1    650  1900
@@
 F 0 "J3" H 650 3200 50  0000 C CNN
 F 1 "OLED2" H 650 2400 50  0000 C CNN
-F 2 "" H 650 2800 50  0001 C CNN
+F 2 "Socket_Strips:Socket_Strip_Straight_1x07" H 650 2800 50  0001 C CNN
 F 3 "" H 650 2800 50  0001 C CNN
 	1    650  2800
@@
 F 0 "J4" H 650 4100 50  0000 C CNN
 F 1 "OLED3" H 650 3300 50  0000 C CNN
-F 2 "" H 650 3700 50  0001 C CNN
+F 2 "Socket_Strips:Socket_Strip_Straight_1x07" H 650 3700 50  0001 C CNN
 F 3 "" H 650 3700 50  0001 C CNN
 	1    650  3700
@@
 F 0 "J5" H 650 5000 50  0000 C CNN
 F 1 "OLED4" H 650 4200 50  0000 C CNN
-F 2 "" H 650 4600 50  0001 C CNN
+F 2 "Socket_Strips:Socket_Strip_Straight_1x07" H 650 4600 50  0001 C CNN
 F 3 "" H 650 4600 50  0001 C CNN
 	1    650  4600
@@
 F 0 "J6" H 650 5900 50  0000 C CNN
 F 1 "OLED5" H 650 5100 50  0000 C CNN
-F 2 "" H 650 5500 50  0001 C CNN
+F 2 "Socket_Strips:Socket_Strip_Straight_1x07" H 650 5500 50  0001 C CNN
 F 3 "" H 650 5500 50  0001 C CNN
 	1    650  5500
@@
 F 0 "J7" H 650 6800 50  0000 C CNN
 F 1 "OLED6" H 650 6000 50  0000 C CNN
-F 2 "" H 650 6400 50  0001 C CNN
+F 2 "Socket_Strips:Socket_Strip_Straight_1x07" H 650 6400 50  0001 C CNN
 F 3 "" H 650 6400 50  0001 C CNN
 	1    650  6400
@@
 F 0 "J8" H 650 7700 50  0000 C CNN
 F 1 "OLED7" H 650 6900 50  0000 C CNN
-F 2 "" H 650 7300 50  0001 C CNN
+F 2 "Socket_Strips:Socket_Strip_Straight_1x07" H 650 7300 50  0001 C CNN
 F 3 "" H 650 7300 50  0001 C CNN
 	1    650  7300
@@
 F 0 "J9" H 9850 2800 50  0000 C CNN
 F 1 "Conn_02x16_Odd_Even" H 9850 1100 50  0000 C CNN
-F 2 "" H 9800 2000 50  0001 C CNN
+F 2 "Pin_Headers:Pin_Header_Straight_2x16" H 9800 2000 50  0001 C CNN
 F 3 "" H 9800 2000 50  0001 C CNN
 	1    9800 2000
@@
 F 0 "U1" H 2450 1250 50  0000 C CNN
 F 1 "74xx238" H 2450 1400 50  0000 C CNN
-F 2 "" H 2450 1250 60  0001 C CNN
+F 2 "Housings_DIP:DIP-16_W7.62mm" H 2450 1250 60  0001 C CNN
 F 3 "" H 2450 1250 60  0001 C CNN
 	1    2450 1300
@@
 F 0 "C1" H 9010 3820 50  0000 L CNN
 F 1 "10nF" H 9010 3670 50  0000 L CNN
-F 2 "" H 9000 3750 50  0001 C CNN
+F 2 "Capacitors_SMD:C_0805_HandSoldering" H 9000 3750 50  0001 C CNN
 F 3 "" H 9000 3750 50  0001 C CNN
 	1    9000 3750
@@
 F 0 "RV4" H 6150 4100 50  0000 C CNN
 F 1 "RSA0N11M9A0J" V 5900 4000 50  0001 C CNN
-F 2 "" H 6000 4000 50  0001 C CNN
+F 2 "ca_alps:AlpsFader_RSA0N11M9A0J" H 6000 4000 50  0001 C CNN
 F 3 "" H 6000 4000 50  0001 C CNN
 	1    6000 4000
@@
 F 0 "U9" H 7850 5650 50  0000 C CNN
 F 1 "74xx238" H 7850 5800 50  0000 C CNN
-F 2 "" H 7850 5650 60  0001 C CNN
+F 2 "Housings_DIP:DIP-16_W7.62mm" H 7850 5650 60  0001 C CNN
 F 3 "" H 7850 5650 60  0001 C CNN
 	1    7850 5700
@@
 F 0 "C11" H 11010 3820 50  0000 L CNN
 F 1 "10nF" H 11010 3670 50  0000 L CNN
-F 2 "" H 11000 3750 50  0001 C CNN
+F 2 "Capacitors_SMD:C_0805_HandSoldering" H 11000 3750 50  0001 C CNN
 F 3 "" H 11000 3750 50  0001 C CNN
 	1    11000 3750
@@
 F 0 "U6" H 7450 3650 60  0000 C CNN
 F 1 "CAP1296" H 7500 2850 60  0000 C CNN
-F 2 "" H 7400 3300 60  0001 C CNN
+F 2 "Housings_DFN_QFN:DFN-10-1EP_3x3mm_Pitch0.5mm" H 7400 3300 60  0001 C CNN
 F 3 "" H 7400 3300 60  0001 C CNN
 	1    7500 3250
@@
 F 0 "U7" H 7450 4700 60  0000 C CNN
 F 1 "CAP1296" H 7500 3900 60  0000 C CNN
-F 2 "" H 7400 4350 60  0001 C CNN
+F 2 "Housings_DFN_QFN:DFN-10-1EP_3x3mm_Pitch0.5mm" H 7400 4350 60  0001 C CNN
 F 3 "" H 7400 4350 60  0001 C CNN
 	1    7500 4300
@@
 F 0 "R1" H 8080 3420 50  0000 L CNN
 F 1 "2k2" H 8080 3360 50  0000 L CNN
-F 2 "" H 8050 3400 50  0001 C CNN
+F 2 "Resistors_SMD:R_1206_HandSoldering" H 8050 3400 50  0001 C CNN
 F 3 "" H 8050 3400 50  0001 C CNN
 	1    8050 3400
@@
 F 0 "R2" H 8080 4470 50  0000 L CNN
 F 1 "2k2" H 8080 4410 50  0000 L CNN
-F 2 "" H 8050 4450 50  0001 C CNN
+F 2 "Resistors_SMD:R_1206_HandSoldering" H 8050 4450 50  0001 C CNN
 F 3 "" H 8050 4450 50  0001 C CNN
 	1    8050 4450

Commit message: Updated component maps ready for board layout, adding Thumbs.db to .gitignore
Parts:
- J1, J2, J3, J4, J5, J6, J7, J8: footprint Socket_Strips:Socket_Strip_Straight_1x07 -> ca_displays:0.95_SPI_SSD1306_Display
- J9: footprint Pin_Headers:Pin_Header_Straight_2x16 -> Pin_Headers:Pin_Header_Angled_2x16_Pitch2.54mm
Changed lines of the file:
@@
 F 0 "J1" H 650 1400 50  0000 C CNN
 F 1 "OLED0" H 650 600 50  0000 C CNN
-F 2 "Socket_Strips:Socket_Strip_Straight_1x07" H 650 1000 50  0001 C CNN
+F 2 "ca_displays:0.95_SPI_SSD1306_Display" H 650 1000 50  0001 C CNN
 F 3 "" H 650 1000 50  0001 C CNN
 	1    650  1000
@@
 F 0 "J2" H 650 2300 50  0000 C CNN
 F 1 "OLED1" H 650 1500 50  0000 C CNN
-F 2 "Socket_Strips:Socket_Strip_Straight_1x07" H 650 1900 50  0001 C CNN
+F 2 "ca_displays:0.95_SPI_SSD1306_Display" H 650 1900 50  0001 C CNN
 F 3 "" H 650 1900 50  0001 C CNN
 	1    650  1900
@@
 F 0 "J3" H 650 3200 50  0000 C CNN
 F 1 "OLED2" H 650 2400 50  0000 C CNN
-F 2 "Socket_Strips:Socket_Strip_Straight_1x07" H 650 2800 50  0001 C CNN
+F 2 "ca_displays:0.95_SPI_SSD1306_Display" H 650 2800 50  0001 C CNN
 F 3 "" H 650 2800 50  0001 C CNN
 	1    650  2800
@@
 F 0 "J4" H 650 4100 50  0000 C CNN
 F 1 "OLED3" H 650 3300 50  0000 C CNN
-F 2 "Socket_Strips:Socket_Strip_Straight_1x07" H 650 3700 50  0001 C CNN
+F 2 "ca_displays:0.95_SPI_SSD1306_Display" H 650 3700 50  0001 C CNN
 F 3 "" H 650 3700 50  0001 C CNN
 	1    650  3700
@@
 F 0 "J5" H 650 5000 50  0000 C CNN
 F 1 "OLED4" H 650 4200 50  0000 C CNN
-F 2 "Socket_Strips:Socket_Strip_Straight_1x07" H 650 4600 50  0001 C CNN
+F 2 "ca_displays:0.95_SPI_SSD1306_Display" H 650 4600 50  0001 C CNN
 F 3 "" H 650 4600 50  0001 C CNN
 	1    650  4600
@@
 F 0 "J6" H 650 5900 50  0000 C CNN
 F 1 "OLED5" H 650 5100 50  0000 C CNN
-F 2 "Socket_Strips:Socket_Strip_Straight_1x07" H 650 5500 50  0001 C CNN
+F 2 "ca_displays:0.95_SPI_SSD1306_Display" H 650 5500 50  0001 C CNN
 F 3 "" H 650 5500 50  0001 C CNN
 	1    650  5500
@@
 F 0 "J7" H 650 6800 50  0000 C CNN
 F 1 "OLED6" H 650 6000 50  0000 C CNN
-F 2 "Socket_Strips:Socket_Strip_Straight_1x07" H 650 6400 50  0001 C CNN
+F 2 "ca_displays:0.95_SPI_SSD1306_Display" H 650 6400 50  0001 C CNN
 F 3 "" H 650 6400 50  0001 C CNN
 	1    650  6400
@@
 F 0 "J8" H 650 7700 50  0000 C CNN
 F 1 "OLED7" H 650 6900 50  0000 C CNN
-F 2 "Socket_Strips:Socket_Strip_Straight_1x07" H 650 7300 50  0001 C CNN
+F 2 "ca_displays:0.95_SPI_SSD1306_Display" H 650 7300 50  0001 C CNN
 F 3 "" H 650 7300 50  0001 C CNN
 	1    650  7300
@@
 F 0 "J9" H 9850 2800 50  0000 C CNN
 F 1 "Conn_02x16_Odd_Even" H 9850 1100 50  0000 C CNN
-F 2 "Pin_Headers:Pin_Header_Straight_2x16" H 9800 2000 50  0001 C CNN
+F 2 "Pin_Headers:Pin_Header_Angled_2x16_Pitch2.54mm" H 9800 2000 50  0001 C CNN
 F 3 "" H 9800 2000 50  0001 C CNN
 	1    9800 2000

Commit message: Updated first cut at board layout
Parts:
- J9: footprint Pin_Headers:Pin_Header_Angled_2x16_Pitch2.54mm -> Pin_Headers:Pin_Header_Straight_2x16_Pitch2.54mm
Changed lines of the file:
@@
 F 0 "J9" H 9850 2800 50  0000 C CNN
 F 1 "Conn_02x16_Odd_Even" H 9850 1100 50  0000 C CNN
-F 2 "Pin_Headers:Pin_Header_Angled_2x16_Pitch2.54mm" H 9800 2000 50  0001 C CNN
+F 2 "Pin_Headers:Pin_Header_Straight_2x16_Pitch2.54mm" H 9800 2000 50  0001 C CNN
 F 3 "" H 9800 2000 50  0001 C CNN
 	1    9800 2000

Commit message: Updated to fix missing power pins for LCDs, updated DFN chips with right pinout
Parts:
- U6, U7: symbol CAP1296 -> CAP1296_DFN
Connections:
- net FCAP0: now also U6.1 (CS1); no longer U6.2 (CS1)
- net FCAP1: now also U6.10 (CS2); no longer U6.13 (CS2)
- net FCAP2: now also U6.9 (CS3); no longer U6.12 (CS3)
- net FCAP3: now also U6.8 (CS4); no longer U6.11 (CS4)
- net FCAP4: now also U7.1 (CS1); no longer U7.2 (CS1)
- net FCAP5: now also U7.10 (CS2); no longer U7.13 (CS2)
- net FCAP6: now also U7.9 (CS3); no longer U7.12 (CS3)
- net FCAP7: now also U7.8 (CS4); no longer U7.11 (CS4)
- net FSCLa: now also U6.4 (SCL); no longer U6.5 (SCL)
- net FSCLb: now also U7.4 (SCL); no longer U7.5 (SCL)
- net FSDAa: now also U6.3 (SDA); no longer U6.4 (SDA)
- net FSDAb: now also U7.3 (SDA); no longer U7.4 (SDA)
- net GND: now also J1.1 (Pin_1), J2.1 (Pin_1), J3.1 (Pin_1), J4.1 (Pin_1), J5.1 (Pin_1), J6.1 (Pin_1), J7.1 (Pin_1), J8.1 (Pin_1), U6.11 (GND), U6.6 (CS6), U6.7 (CS5), U7.11 (GND), U7.6 (CS6), U7.7 (CS5); no longer U6.10 (CS5), U6.8 (GND), U6.9 (CS6), U7.10 (CS5), U7.8 (GND), U7.9 (CS6)
- net VCC: now also J1.2 (Pin_2), J2.2 (Pin_2), J3.2 (Pin_2), J4.2 (Pin_2), J5.2 (Pin_2), J6.2 (Pin_2), J7.2 (Pin_2), J8.2 (Pin_2), U6.5 (VDD), U7.5 (VDD); no longer U6.7 (VDD), U7.7 (VDD)
- net at R1.1: now also U6.2 (INT); no longer U6.3 (INT)
- net at R2.1: now also U7.2 (INT); no longer U7.3 (INT)
Changed lines of the file:
@@
 Connection ~ 1000 5200
 Wire Wire Line
-	1000 7000 850  7000
+	850  7000 1600 7000
 Connection ~ 1000 6100
 Wire Wire Line
@@
 Wire Wire Line
 	10100 1600 10400 1600
-Wire Wire Line
-	10100 1800 10400 1800
 Wire Wire Line
 	10100 1900 10400 1900
@@
 Connection ~ 10750 3950
 $Comp
-L CAP1296 U6
+L CAP1296_DFN U6
 U 1 1 5A6E4F8D
 P 7500 3250
@@
 $EndComp
 $Comp
-L CAP1296 U7
+L CAP1296_DFN U7
 U 1 1 5A6E5698
 P 7500 4300
@@
 	9600 1600 9350 1600
 Connection ~ 8850 1800
+$Comp
+L GND #PWR026
+U 1 1 5AFD5D40
+P 1600 7100
+F 0 "#PWR026" H 1600 6850 50  0001 C CNN
+F 1 "GND" H 1600 6950 50  0000 C CNN
+F 2 "" H 1600 7100 50  0001 C CNN
+F 3 "" H 1600 7100 50  0001 C CNN
+	1    1600 7100
+	1    0    0    -1
+$EndComp
+$Comp
+L VCC #PWR027
+U 1 1 5AFD5E9C
+P 1600 6800
+F 0 "#PWR027" H 1600 6650 50  0001 C CNN
+F 1 "VCC" H 1600 6950 50  0000 C CNN
+F 2 "" H 1600 6800 50  0001 C CNN
+F 3 "" H 1600 6800 50  0001 C CNN
+	1    1600 6800
+	1    0    0    -1
+$EndComp
+Wire Wire Line
+	1600 7000 1600 7100
+Connection ~ 1000 7000
+Wire Wire Line
+	1600 6800 1600 6900
+Wire Wire Line
+	1600 6900 950  6900
+Connection ~ 950  6900
+Wire Wire Line
+	10100 1800 10400 1800
 $EndSCHEMATC

Commit message: Adding DIP library for DIP to DFN converter, Updated board layout with autorouting, hopefully v0.1 final design
Parts:
- C1, C10, C11, C12, C13, C2, C3, C4, C5, C6, C7, C8, C9: footprint Capacitors_SMD:C_0805_HandSoldering -> Capacitors_THT:C_Disc_D5.0mm_W2.5mm_P5.00mm
- R1, R2: footprint Resistors_SMD:R_1206_HandSoldering -> Resistors_THT:R_Axial_DIN0204_L3.6mm_D1.6mm_P5.08mm_Horizontal
Changed lines of the file:
@@
 F 0 "C2" H 9260 3820 50  0000 L CNN
 F 1 "10nF" H 9260 3670 50  0000 L CNN
-F 2 "Capacitors_SMD:C_0805_HandSoldering" H 9250 3750 50  0001 C CNN
+F 2 "Capacitors_THT:C_Disc_D5.0mm_W2.5mm_P5.00mm" H 9250 3750 50  0001 C CNN
 F 3 "" H 9250 3750 50  0001 C CNN
 	1    9250 3750
@@
 F 0 "C3" H 9510 3820 50  0000 L CNN
 F 1 "10nF" H 9510 3670 50  0000 L CNN
-F 2 "Capacitors_SMD:C_0805_HandSoldering" H 9500 3750 50  0001 C CNN
+F 2 "Capacitors_THT:C_Disc_D5.0mm_W2.5mm_P5.00mm" H 9500 3750 50  0001 C CNN
 F 3 "" H 9500 3750 50  0001 C CNN
 	1    9500 3750
@@
 F 0 "C4" H 9760 3820 50  0000 L CNN
 F 1 "10nF" H 9760 3670 50  0000 L CNN
-F 2 "Capacitors_SMD:C_0805_HandSoldering" H 9750 3750 50  0001 C CNN
+F 2 "Capacitors_THT:C_Disc_D5.0mm_W2.5mm_P5.00mm" H 9750 3750 50  0001 C CNN
 F 3 "" H 9750 3750 50  0001 C CNN
 	1    9750 3750
@@
 F 0 "C5" H 10010 3820 50  0000 L CNN
 F 1 "10nF" H 10010 3670 50  0000 L CNN
-F 2 "Capacitors_SMD:C_0805_HandSoldering" H 10000 3750 50  0001 C CNN
+F 2 "Capacitors_THT:C_Disc_D5.0mm_W2.5mm_P5.00mm" H 10000 3750 50  0001 C CNN
 F 3 "" H 10000 3750 50  0001 C CNN
 	1    10000 3750
@@
 F 0 "C6" H 10260 3820 50  0000 L CNN
 F 1 "10nF" H 10260 3670 50  0000 L CNN
-F 2 "Capacitors_SMD:C_0805_HandSoldering" H 10250 3750 50  0001 C CNN
+F 2 "Capacitors_THT:C_Disc_D5.0mm_W2.5mm_P5.00mm" H 10250 3750 50  0001 C CNN
 F 3 "" H 10250 3750 50  0001 C CNN
 	1    10250 3750
@@
 F 0 "C7" H 10510 3820 50  0000 L CNN
 F 1 "10nF" H 10510 3670 50  0000 L CNN
-F 2 "Capacitors_SMD:C_0805_HandSoldering" H 10500 3750 50  0001 C CNN
+F 2 "Capacitors_THT:C_Disc_D5.0mm_W2.5mm_P5.00mm" H 10500 3750 50  0001 C CNN
 F 3 "" H 10500 3750 50  0001 C CNN
 	1    10500 3750
@@
 F 0 "C10" H 10760 3820 50  0000 L CNN
 F 1 "10nF" H 10760 3670 50  0000 L CNN
-F 2 "Capacitors_SMD:C_0805_HandSoldering" H 10750 3750 50  0001 C CNN
+F 2 "Capacitors_THT:C_Disc_D5.0mm_W2.5mm_P5.00mm" H 10750 3750 50  0001 C CNN
 F 3 "" H 10750 3750 50  0001 C CNN
 	1    10750 3750
@@
 F 0 "C8" H 10510 4620 50  0000 L CNN
 F 1 "10nF" H 10510 4470 50  0000 L CNN
-F 2 "Capacitors_SMD:C_0805_HandSoldering" H 10500 4550 50  0001 C CNN
+F 2 "Capacitors_THT:C_Disc_D5.0mm_W2.5mm_P5.00mm" H 10500 4550 50  0001 C CNN
 F 3 "" H 10500 4550 50  0001 C CNN
 	1    10500 4550
@@
 F 0 "C12" H 11010 4620 50  0000 L CNN
 F 1 "10nF" H 11010 4470 50  0000 L CNN
-F 2 "Capacitors_SMD:C_0805_HandSoldering" H 11000 4550 50  0001 C CNN
+F 2 "Capacitors_THT:C_Disc_D5.0mm_W2.5mm_P5.00mm" H 11000 4550 50  0001 C CNN
 F 3 "" H 11000 4550 50  0001 C CNN
 	1    11000 4550
@@
 F 0 "C9" H 10510 5720 50  0000 L CNN
 F 1 "10nF" H 10510 5570 50  0000 L CNN
-F 2 "Capacitors_SMD:C_0805_HandSoldering" H 10500 5650 50  0001 C CNN
+F 2 "Capacitors_THT:C_Disc_D5.0mm_W2.5mm_P5.00mm" H 10500 5650 50  0001 C CNN
 F 3 "" H 10500 5650 50  0001 C CNN
 	1    10500 5650
@@
 F 0 "C13" H 11010 5720 50  0000 L CNN
 F 1 "10nF" H 11010 5570 50  0000 L CNN
-F 2 "Capacitors_SMD:C_0805_HandSoldering" H 11000 5650 50  0001 C CNN
+F 2 "Capacitors_THT:C_Disc_D5.0mm_W2.5mm_P5.00mm" H 11000 5650 50  0001 C CNN
 F 3 "" H 11000 5650 50  0001 C CNN
 	1    11000 5650
@@
 F 0 "C1" H 9010 3820 50  0000 L CNN
 F 1 "10nF" H 9010 3670 50  0000 L CNN
-F 2 "Capacitors_SMD:C_0805_HandSoldering" H 9000 3750 50  0001 C CNN
+F 2 "Capacitors_THT:C_Disc_D5.0mm_W2.5mm_P5.00mm" H 9000 3750 50  0001 C CNN
 F 3 "" H 9000 3750 50  0001 C CNN
 	1    9000 3750
@@
 F 0 "C11" H 11010 3820 50  0000 L CNN
 F 1 "10nF" H 11010 3670 50  0000 L CNN
-F 2 "Capacitors_SMD:C_0805_HandSoldering" H 11000 3750 50  0001 C CNN
+F 2 "Capacitors_THT:C_Disc_D5.0mm_W2.5mm_P5.00mm" H 11000 3750 50  0001 C CNN
 F 3 "" H 11000 3750 50  0001 C CNN
 	1    11000 3750
@@
 F 0 "R1" H 8080 3420 50  0000 L CNN
 F 1 "2k2" H 8080 3360 50  0000 L CNN
-F 2 "Resistors_SMD:R_1206_HandSoldering" H 8050 3400 50  0001 C CNN
+F 2 "Resistors_THT:R_Axial_DIN0204_L3.6mm_D1.6mm_P5.08mm_Horizontal" H 8050 3400 50  0001 C CNN
 F 3 "" H 8050 3400 50  0001 C CNN
 	1    8050 3400
@@
 F 0 "R2" H 8080 4470 50  0000 L CNN
 F 1 "2k2" H 8080 4410 50  0000 L CNN
-F 2 "Resistors_SMD:R_1206_HandSoldering" H 8050 4450 50  0001 C CNN
+F 2 "Resistors_THT:R_Axial_DIN0204_L3.6mm_D1.6mm_P5.08mm_Horizontal" H 8050 4450 50  0001 C CNN
 F 3 "" H 8050 4450 50  0001 C CNN
 	1    8050 4450

Commit message: Added prototype label
Other:
- note added: "PROTOTYPE BOARD (NO LONGER CURRENT)"
Changed lines of the file:
@@
 Wire Wire Line
 	10100 1800 10400 1800
+Text Notes 5100 950  0    60   ~ 0
+PROTOTYPE BOARD (NO LONGER CURRENT)
 $EndSCHEMATC
