File: hardware/board-x8-fader-display/board-x8-fader-display.sch (KiCad schematic (older format))
At the start: 40 parts, among them J1 OLED0, J2 OLED1, J3 OLED2, J4 OLED3, J5 OLED4, J6 OLED5, J7 OLED6, J8 OLED7, J9 Conn_02x16_Odd_Even, U1 74xx138, U10 74xx238, U2 74xx138, U3 L293, U4 L293, U5 L293, U6 L293, U7 CAP1296, U8 CAP1296, U9 4051

Commit message: Updating PCB and schema for ProtoAdvantage DIP to DFN adapter (not great but easier than SMD on this board). Rerouting and manual edits to conform to DRC / track & pad clearance
Parts:
- U7, U8: symbol CAP1296_DFN -> CAP1296_PROTOADV_DFNTODIP
Connections:
- net +12V: now also J9.4 (Pin_4)
- net GND: no longer J9.4 (Pin_4)
Changed lines of the file:
@@
 	10100 1300 10900 1300
-Wire Wire Line
-	10100 1400 10900 1400
 Wire Wire Line
 	10100 1500 11050 1500
@@
 $EndComp
 $Comp
-L GND #PWR015
-U 1 1 5A6E9588
-P 10900 2850
-F 0 "#PWR015" H 10900 2600 50  0001 C CNN
-F 1 "GND" H 10900 2700 50  0000 C CNN
-F 2 "" H 10900 2850 50  0001 C CNN
-F 3 "" H 10900 2850 50  0001 C CNN
-	1    10900 2850
-	1    0    0    -1
-$EndComp
-$Comp
 L VCC #PWR016
 U 1 1 5A6E962D
@@
 	11050 1500 11050 1000
 Wire Wire Line
-	10900 1400 10900 2850
-Wire Wire Line
 	8750 1150 8750 1400
 Text Label 9350 1300 0    60   ~ 0
@@
 GND
 Text Label 10400 1400 2    60   ~ 0
-GND
+Vmotor
 Text Label 10400 1300 2    60   ~ 0
 VCC
@@
 Connection ~ 10500 3950
 $Comp
-L CAP1296_DFN U7
+L CAP1296_PROTOADV_DFNTODIP U7
 U 1 1 5A6E4F8D
 P 7500 3250
@@
 $EndComp
 $Comp
-L CAP1296_DFN U8
+L CAP1296_PROTOADV_DFNTODIP U8
 U 1 1 5A6E5698
 P 7500 4300
@@
 Wire Wire Line
 	7950 4350 8150 4350
-Wire Wire Line
-	7000 4450 7000 4800
 Wire Wire Line
 	7000 4450 7050 4450
@@
 Wire Wire Line
 	4850 4700 4850 4650
-Text Label 7000 3750 1    60   ~ 0
-SMDGND
-Text Label 7000 4800 1    60   ~ 0
-SMDGND
-Wire Wire Line
-	7000 3400 7000 3750
+Text Label 7000 3600 1    60   ~ 0
+GND
+Text Label 7000 4650 1    60   ~ 0
+GND
 $Comp
 L GND #PWR025
 U 1 1 5B135741
-P 9750 4500
-F 0 "#PWR025" H 9750 4250 50  0001 C CNN
-F 1 "GND" H 9750 4350 50  0000 C CNN
-F 2 "" H 9750 4500 50  0001 C CNN
-F 3 "" H 9750 4500 50  0001 C CNN
-	1    9750 4500
-	1    0    0    -1
-$EndComp
-Wire Wire Line
-	9750 4500 9750 4400
-Wire Wire Line
-	9750 4400 9400 4400
-Text Label 9400 4400 0    60   ~ 0
-SMDGND
+P 7000 4700
+F 0 "#PWR025" H 7000 4450 50  0001 C CNN
+F 1 "GND" H 7000 4550 50  0000 C CNN
+F 2 "" H 7000 4700 50  0001 C CNN
+F 3 "" H 7000 4700 50  0001 C CNN
+	1    7000 4700
+	1    0    0    -1
+$EndComp
+$Comp
+L GND #PWR026
+U 1 1 5B1CCAC3
+P 7000 3650
+F 0 "#PWR026" H 7000 3400 50  0001 C CNN
+F 1 "GND" H 7000 3500 50  0000 C CNN
+F 2 "" H 7000 3650 50  0001 C CNN
+F 3 "" H 7000 3650 50  0001 C CNN
+	1    7000 3650
+	1    0    0    -1
+$EndComp
+Wire Wire Line
+	7000 4450 7000 4700
+Wire Wire Line
+	7000 3400 7000 3650
+Wire Wire Line
+	10100 1400 11050 1400
+Connection ~ 11050 1400
 $EndSCHEMATC
