File: hardware/board-controller-2560hat/board-controller-2560hat.sch (KiCad schematic (older format))
At the start: 20 parts, among them J1 Conn_02x16_Odd_Even, J2 Conn_02x16_Odd_Even, J3 Conn_02x16_Odd_Even, J4 Conn_01x08, J5 Conn_02x16_Odd_Even, U1 74HC4050DTSSOP, U2 TCA9548A_TSSOP, U3 RFM69HCW_SMT, X1 SMACONNECTOR_EDGE

Commit message: Adding component libraries and docs for keypad and LED drivers. Still need to add TFT before complete
Parts:
- added D1, D10, D11, D12, D13, D14, D15, D16, D2, D3, D4, D5, D6, D7, D8, D9: LED, symbol LED
- added R1, R2: 2k2, _1206, symbol RESISTOR_1206
- added RN3, RN4: 750R, symbol R_Pack08
- added SW1, SW10, SW11, SW12, SW13, SW14, SW15, SW16, SW2, SW3, SW4, SW5, SW6, SW7, SW8, SW9: SW_Push_45deg, symbol SW_Push_45deg
- added U4: PCF8574, symbol PCF8574
- added U5: PCA9635PW, SOP65P640X110-28N, symbol PCA9635PW
- J1: value Conn_02x16_Odd_Even -> CONN_BOARD0
- J2: value Conn_02x16_Odd_Even -> CONN_BOARD1
- J3: value Conn_02x16_Odd_Even -> CONN_BOARD2
- J4: value Conn_01x08 -> CONN_POWER
- J5: value Conn_02x16_Odd_Even -> CONN_BOARD3
- renumbered U2 to U1, U1 to U2
Connections:
- net +5V: now also R1.2, R2.2, RN3.10 (R7.2), RN3.11 (R6.2), RN3.12 (R5.2), RN3.13 (R4.2), RN3.14 (R3.2), RN3.15 (R2.2), RN3.16 (R1.2), RN3.9 (R8.2), RN4.1 (R1.1), RN4.2 (R2.1), RN4.3 (R3.1), RN4.4 (R4.1), RN4.5 (R5.1), RN4.6 (R6.1), RN4.7 (R7.1), RN4.8 (R8.1), U4.16 (VDD), U5.1 (A0), U5.2 (A1), U5.28 (VDD)
- net GND: now also U4.1 (A0), U4.2 (A1), U4.3 (A2), U4.8 (VSS), U5.14 (VSS), U5.23 (~OE), U5.24 (A5), U5.25 (A6), U5.3 (A2), U5.4 (A3), U5.5 (A4)
- net RFM_RST_5v: now also XA1.D47; no longer XA1.D2 (D2_INT0)
- net MUX_SCL renamed SCL
- net SCL: now also R1.1, U4.14 (SCL), U5.26 (SCL)
- net MUX_SDA renamed SDA
- net SDA: now also R2.1, U4.15 (SDA), U5.27 (SDA)
- new net: D8.1 (K), U5.10 (LED4)
- new net: D13.1 (K), U5.11 (LED5)
- new net: D3.1 (K), U5.12 (LED6)
- new net: D9.1 (K), U5.13 (LED7)
- new net: D14.1 (K), U5.15 (LED8)
- new net: D4.1 (K), U5.16 (LED9)
- new net: D10.1 (K), U5.17 (LED10)
- new net: D15.1 (K), U5.18 (LED11)
- new net: D5.1 (K), U5.19 (LED12)
- new net: D11.1 (K), U5.20 (LED13)
- new net: D16.1 (K), U5.21 (LED14)
- new net: D6.1 (K), U5.22 (LED15)
- new net: D1.1 (K), U5.6 (LED0)
- new net: D7.1 (K), U5.7 (LED1)
- new net: D12.1 (K), U5.8 (LED2)
- new net: D2.1 (K), U5.9 (LED3)
- new net: D1.2 (A), RN3.1 (R1.1)
- new net: SW1.1, SW13.1, SW5.1, SW9.1, U4.4 (P0)
- new net: SW1.2, SW2.2, SW3.2, SW4.2, U4.9 (P4)
- new net: D7.2 (A), RN3.2 (R2.1)
- new net: D12.2 (A), RN3.3 (R3.1)
- new net: D2.2 (A), RN3.4 (R4.1)
- new net: D8.2 (A), RN3.5 (R5.1)
- new net: D13.2 (A), RN3.6 (R6.1)
- new net: D3.2 (A), RN3.7 (R7.1)
- new net: D9.2 (A), RN3.8 (R8.1)
- new net: D14.2 (A), RN4.9 (R8.2)
- new net: D4.2 (A), RN4.10 (R7.2)
- new net: D10.2 (A), RN4.11 (R6.2)
- new net: D15.2 (A), RN4.12 (R5.2)
- new net: D5.2 (A), RN4.13 (R4.2)
- new net: D11.2 (A), RN4.14 (R3.2)
- new net: D16.2 (A), RN4.15 (R2.2)
- new net: D6.2 (A), RN4.16 (R1.2)
- new net: SW5.2, SW6.2, SW7.2, SW8.2, U4.10 (P5)
- new net: SW10.2, SW11.2, SW12.2, SW9.2, U4.11 (P6)
- new net: SW13.2, SW14.2, SW15.2, SW16.2, U4.12 (P7)
- new net: SW10.1, SW14.1, SW2.1, SW6.1, U4.5 (P1)
- new net: SW11.1, SW15.1, SW3.1, SW7.1, U4.6 (P2)
- new net: SW12.1, SW16.1, SW4.1, SW8.1, U4.7 (P3)
- new net KBD_~INT~: U4.13 (~INT~), XA1.D2 (D2_INT0)
- no-connect marks 34 -> 33
Other:
- note added: "4x4 LED illuminated Keypad"
- note added: "Fader Touch capacitive sensor demux"
- note added: "Radio module"
- moved on the sheet: C1, C2, C3, C4, C5, C6, C7, C8, J1, J2, J3, J4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

Commit message: Fixing TFT_ pinouts and rebuilding PCB
Parts:
- removed D1, D10, D11, D12, D13, D14, D15, D16, D2, D3, D4, D5, D6, D7, D8, D9: LED, symbol LED
- removed RN3, RN4: 750R, symbol R_Pack08
- removed SW1, SW10, SW11, SW12, SW13, SW14, SW15, SW16, SW2, SW3, SW4, SW5, SW6, SW7, SW8, SW9: SW_Push_45deg, symbol SW_Push_45deg
- added J2: CONN_LCD, Pin_Headers:Pin_Header_Straight_2x08_Pitch2.54mm, symbol Conn_02x08_Odd_Even
- added J7: CONN_SW, Connectors_Terminal_Blocks:TerminalBlock_Pheonix_MPT-2.54mm_4pol, symbol Screw_Terminal_01x04
- added J8: CONN_KEYLED, Pin_Headers:Pin_Header_Straight_1x18_Pitch2.54mm, symbol Conn_01x18
- added J9: CONN_KEYSW, Pin_Headers:Pin_Header_Straight_1x08_Pitch2.54mm, symbol Conn_01x08
- C1, C2, C3, C4, C5, C6, C7, C8: footprint _0603 -> Capacitors_SMD:C_0603_HandSoldering
- J1: renamed from J4; footprint (none) -> Pin_Headers:Pin_Header_Straight_1x08_Pitch2.54mm
- J3: renamed from J1; footprint (none) -> Pin_Headers:Pin_Header_Straight_2x16_Pitch2.54mm
- J4: renamed from J2; footprint (none) -> Pin_Headers:Pin_Header_Straight_2x16_Pitch2.54mm
- J5: renamed from J3; footprint (none) -> Pin_Headers:Pin_Header_Straight_2x16_Pitch2.54mm
- J6: renamed from J5; footprint (none) -> Pin_Headers:Pin_Header_Straight_2x16_Pitch2.54mm
- R1, R2: footprint _1206 -> Capacitors_SMD:C_1206_HandSoldering
- RN3: renamed from RN1; footprint (none) -> Housings_SOIC:CA_SOIC_16_5.59x11.18_1.27_Pitch
- RN4: renamed from RN2; footprint (none) -> Housings_SOIC:CA_SOIC_16_5.59x11.18_1.27_Pitch
- U1: renamed from U2; footprint TSSOP16 -> Housings_SSOP:SSOP-16_5.3x6.2mm_Pitch0.65mm
- U2: renamed from U3; footprint RFMHCW_SMT -> Adafruit RFM+LoRa Breakout:RFMHCW_SMT
- U3: renamed from U4; footprint (none) -> Housings_SOIC:CA_SOIC_16_7.5x10.5_1.27_Pitch
- U4: renamed from U5; footprint SOP65P640X110-28N -> Housings_SSOP:TSSOP-28_4.4x9.7mm_Pitch0.65mm
- X1: footprint SMA_EDGELAUNCH -> Adafruit RFM+LoRa Breakout:SMA_EDGELAUNCH
- XA1: footprint (none) -> Arduino:Arduino_Mega2560_Shield
- renumbered U1 to U5
Connections:
- net +3.3v is gone; now on net +3V3: J1.5 (Pin_5)
- net Vcc is gone; now on net +5V: J3.2 (Pin_2), J4.2 (Pin_2), J5.2 (Pin_2), J6.2 (Pin_2)
- net Vmotor is gone; now on net +9V: J3.4 (Pin_4), J3.6 (Pin_6), J4.4 (Pin_4), J4.6 (Pin_6), J5.4 (Pin_4), J5.6 (Pin_6), J6.4 (Pin_4), J6.6 (Pin_6)
- net +5V: now also J2.1 (Pin_1), J8.17 (Pin_17), J8.18 (Pin_18)
- net +9V: now also J7.3 (Pin_3)
- net DSCL: now also J2.3 (Pin_3)
- net DSDA: now also J2.5 (Pin_5)
- net GND: now also J2.11 (Pin_11), J2.13 (Pin_13), J2.15 (Pin_15), J2.2 (Pin_2), J2.9 (Pin_9), J7.2 (Pin_2); no longer XA1.A12, XA1.A13, XA1.A14, XA1.A15
- net ~RESET~: now also J7.1 (Pin_1)
- net LCD_LITE: now reaches XA1.D10
- net LCD_LITE: now also J2.4 (Pin_4)
- net LCD_D~C~: now reaches XA1.D11
- net LCD_D~C~: now also J2.8 (Pin_8)
- net LCD_~CS~: now reaches XA1.D12
- net LCD_~CS~: now also J2.7 (Pin_7)
- net LCD_~RST~: now reaches XA1.D13
- net LCD_~RST~: now also J2.6 (Pin_6)
- net KEY_LED4: now reaches U4.10 (LED4)
- net KEY_LED4: now also J8.5 (Pin_5)
- net KEY_LED5: now reaches U4.11 (LED5)
- net KEY_LED5: now also J8.6 (Pin_6)
- net KEY_LED6: now reaches U4.12 (LED6)
- net KEY_LED6: now also J8.7 (Pin_7)
- net KEY_LED7: now reaches U4.13 (LED7)
- net KEY_LED7: now also J8.8 (Pin_8)
- net KEY_LED8: now reaches U4.15 (LED8)
- net KEY_LED8: now also J8.9 (Pin_9)
- net KEY_LED9: now reaches U4.16 (LED9)
- net KEY_LED9: now also J8.10 (Pin_10)
- net KEY_LED10: now reaches U4.17 (LED10)
- net KEY_LED10: now also J8.11 (Pin_11)
- net KEY_LED11: now reaches U4.18 (LED11)
- net KEY_LED11: now also J8.12 (Pin_12)
- net KEY_LED12: now reaches U4.19 (LED12)
- net KEY_LED12: now also J8.13 (Pin_13)
- net KEY_LED13: now reaches U4.20 (LED13)
- net KEY_LED13: now also J8.14 (Pin_14)
- net KEY_LED14: now reaches U4.21 (LED14)
- net KEY_LED14: now also J8.15 (Pin_15)
- net KEY_LED15: now reaches U4.22 (LED15)
- net KEY_LED15: now also J8.16 (Pin_16)
- net KEY_LED0: now reaches U4.6 (LED0)
- net KEY_LED0: now also J8.1 (Pin_1)
- net KEY_LED1: now reaches U4.7 (LED1)
- net KEY_LED1: now also J8.2 (Pin_2)
- net KEY_LED2: now reaches U4.8 (LED2)
- net KEY_LED2: now also J8.3 (Pin_3)
- net KEY_LED3: now reaches U4.9 (LED3)
- net KEY_LED3: now also J8.4 (Pin_4)
- net KEY_COL0: now reaches U3.4 (P0)
- net KEY_COL0: now also J9.1 (Pin_1)
- net KEY_ROW0: now reaches U3.9 (P4)
- net KEY_ROW0: now also J9.5 (Pin_5)
- net KEY_ROW1: now reaches U3.10 (P5)
- net KEY_ROW1: now also J9.6 (Pin_6)
- net KEY_ROW2: now reaches U3.11 (P6)
- net KEY_ROW2: now also J9.7 (Pin_7)
- net KEY_ROW3: now reaches U3.12 (P7)
- net KEY_ROW3: now also J9.8 (Pin_8)
- net KEY_COL1: now reaches U3.5 (P1)
- net KEY_COL1: now also J9.2 (Pin_2)
- net KEY_COL2: now reaches U3.6 (P2)
- net KEY_COL2: now also J9.3 (Pin_3)
- net KEY_COL3: now reaches U3.7 (P3)
- net KEY_COL3: now also J9.4 (Pin_4)
- net +9v: no longer names the net of J1.1 (Pin_1)
- net +9v: now also J7.4 (Pin_4)
- net RFM_RST_3v3 renamed RFM_~RST~_3v3
- net RFM_RST_5v renamed RFM_~RST~_5v
- new net LCD_X+: J2.12 (Pin_12), XA1.A13
- new net LCD_X-: J2.16 (Pin_16), XA1.A15
- new net LCD_Y+: J2.10 (Pin_10), XA1.A12
- new net LCD_Y-: J2.14 (Pin_14), XA1.A14
- no-connect marks 33 -> 29
Other:
- note added: "(SPI_MISO)"
- note added: "(SPI_MOSI)"
- note added: "(SPI_SCK)"
- moved on the sheet: C1, C2, C3, C4, C5, C6, C7, C8, J1, R2
